Commit message: added 2nd version of hyperdog

File: hyperdog_robot_description/urdf/hyperdog_v2.urdf (robot description, URDF)
Before this commit: robot meshes/hyperdog_v2, 13 links, 12 joints
Links:
- link base_link: mass 3 -> 5; geometry collision mesh filename=../meshes/hyperdog_v2/BodyV2.stl scale=0.001 0.001 0.001; visual mesh filename=../meshes/hyperdog_v2/BodyV2.stl scale=0.001 0.001 0.001
Joints:
- joint BL_hip_joint: origin xyz=-0.175 0.066 0 rpy=0 0 0 -> xyz=-0.19575 0.066 0 rpy=0 0 0
- joint BR_hip_joint: origin xyz=-0.175 -0.066 0 rpy=0 0 0 -> xyz=-0.19575 -0.066 0 rpy=0 0 0
- joint FL_hip_joint: origin xyz=0.175 0.066 0 rpy=0 0 0 -> xyz=0.19575 0.066 0 rpy=0 0 0
- joint FR_hip_joint: origin xyz=0.175 -0.066 0 rpy=0 0 0 -> xyz=0.19575 -0.066 0 rpy=0 0 0
